Commit message: 添加imu

File: install/sam_bot_odom_py/share/sam_bot_odom_py/urdf/sam_bot.urdf (robot description, URDF)
Before this commit: robot mycar, 8 links, 7 joints
Links:
- added link imu_link; visual box size=0.045 0.04 0.012
Joints:
- added joint imu_joint: type fixed, parent base_link, child imu_link, origin xyz=0.0 0.0 0.046 rpy=0 0.0 0.0

Commit message: urdf

File: install/sam_bot_odom_py/share/sam_bot_odom_py/urdf/sam_bot.urdf (robot description, URDF)
Before this commit: robot mycar, 9 links, 8 joints
Joints:
- joint imu_joint: origin xyz=0.0 0.0 0.046 rpy=0 0.0 0.0 -> xyz=0.02 -0.09 0.046 rpy=0 0.0 0.0
